File: Helios_12S_Servo_5V2_Buck.kicad_sch (KiCad schematic)
At the start: 25 parts, among them J1 XT30-PWR-F, J2 XT30-PWR-M, U1 LM65680RZYR

Commit message: Update production files
Parts:
- C6, C7, C8: LCSC C77058 -> C15725
- R1: LCSC C49652939 -> C25741
Changed lines of the file:
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@@
 			)
 		)
-		(property "Datasheet" "https://www.lcsc.com/datasheet/C77058.pdf"
+		(property "Datasheet" "https://www.lcsc.com/datasheet/C15725.pdf"
 			(at 182.88 107.95 0)
 			(hide yes)
@@
 			)
 		)
-		(property "LCSC" "C77058"
+		(property "LCSC" "C15725"
 			(at 182.88 107.95 0)
 			(hide yes)
@@
 			)
 		)
-		(property "Datasheet" "https://www.lcsc.com/datasheet/C77058.pdf"
+		(property "Datasheet" "https://www.lcsc.com/datasheet/C15725.pdf"
 			(at 111.76 80.01 0)
 			(hide yes)
@@
 			)
 		)
-		(property "LCSC" "C77058"
+		(property "LCSC" "C15725"
 			(at 111.76 80.01 0)
 			(hide yes)
@@
 			)
 		)
-		(property "Datasheet" "https://www.lcsc.com/datasheet/C77058.pdf"
+		(property "Datasheet" "https://www.lcsc.com/datasheet/C15725.pdf"
 			(at 96.52 80.01 0)
 			(hide yes)
@@
 			)
 		)
-		(property "LCSC" "C77058"
+		(property "LCSC" "C15725"
 			(at 96.52 80.01 0)
 			(hide yes)
@@
 			)
 		)
-		(property "Datasheet" "https://www.lcsc.com/datasheet/C49652939.pdf"
+		(property "Datasheet" "https://www.lcsc.com/datasheet/C25741.pdf"
 			(at 256.54 119.38 0)
 			(hide yes)
@@
 			)
 		)
-		(property "LCSC" "C49652939"
+		(property "LCSC" "C25741"
 			(at 256.54 119.38 0)
 			(hide yes)
