File: Helios_12S_Servo_5V2_Buck.kicad_pcb (KiCad board)
At the start: 4 copper layers, 64 x 16.5 mm, 25 parts, among them J1 XT30-PWR-F, J2 XT30-PWR-M, U1 LM65680RZYR

Commit message: Update layout/routing
Parts:
- moved C7 8.85 mm to (129.2, 66.6)
- moved C8 5.92 mm to (124.3, 73.8), turned to -90 degrees
- moved U1 4.50 mm to (125.7, 65.4)
- moved C13 4.32 mm to (122.1, 63.4)
- moved C6 3.77 mm to (122.1, 66.7)
- moved R2 3.42 mm to (135.3, 64.6), turned to 0 degrees
- moved C14 3.26 mm to (134.1, 66.9)
- moved R1 3.26 mm to (132.9, 66.9)
- moved C11 2.70 mm to (133.7, 72.0)
- moved C12 2.70 mm to (133.7, 68.4)
- moved TP1 2.30 mm to (131.7, 62.8)
- moved C10 1.50 mm to (132.5, 75.8)
- moved C9 1.30 mm to (137.3, 75.8)
- moved L1 0.70 mm to (130.9, 73.0)
- moved C15 0.70 mm to (117.7, 72.8)
Routing:
- net +BATT: track 16.8 -> 6.96 mm, vias 11 -> 17
- net +5V2: track 13.8 -> 6.50 mm
- net GND: track 9.06 -> 6.28 mm, vias 53 -> 50
- net Net-(U1-PG): track 3.45 -> 5.53 mm
- net /BUCK_BST: track 8.76 -> 10.5 mm
- net /BUCK_FB: track 13.2 -> 13.5 mm, vias 3 -> 2

Commit message: Update layout/routing + production files
Routing:
- net GND: track 6.28 -> 8.83 mm, vias 50 -> 68
Changed lines of the file:
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@@
 			)
 		)
-		(property "Datasheet" "https://www.lcsc.com/datasheet/C77058.pdf"
+		(property "Datasheet" "https://www.lcsc.com/datasheet/C15725.pdf"
 			(at 0 0 90)
 			(layer "F.Fab")
@@
 			)
 		)
-		(property "LCSC" "C77058"
+		(property "LCSC" "C15725"
 			(at 0 0 90)
 			(unlocked yes)
@@
 			)
 		)
-		(property "Datasheet" "https://www.lcsc.com/datasheet/C77058.pdf"
+		(property "Datasheet" "https://www.lcsc.com/datasheet/C15725.pdf"
 			(at 0 0 90)
 			(layer "F.Fab")
@@
 			)
 		)
-		(property "LCSC" "C77058"
+		(property "LCSC" "C15725"
 			(at 0 0 90)
 			(unlocked yes)
@@
 			)
 		)
-		(property "Datasheet" "https://www.lcsc.com/datasheet/C49652939.pdf"
+		(property "Datasheet" "https://www.lcsc.com/datasheet/C25741.pdf"
 			(at 0 0 90)
 			(layer "F.Fab")
@@
 			)
 		)
-		(property "LCSC" "C49652939"
+		(property "LCSC" "C25741"
 			(at 0 0 90)
 			(unlocked yes)
@@
 			)
 		)
-		(property "Datasheet" "https://www.lcsc.com/datasheet/C77058.pdf"
+		(property "Datasheet" "https://www.lcsc.com/datasheet/C15725.pdf"
 			(at 0 0 90)
 			(layer "F.Fab")
@@
 			)
 		)
-		(property "LCSC" "C77058"
+		(property "LCSC" "C15725"
 			(at 0 0 270)
 			(unlocked yes)
@@
 	)
 	(segment
-		(start 121.175 67.475)
+		(start 121.625 67.475)
 		(end 122.1 67.475)
-		(width 0.2)
+		(width 0.3)
 		(layer "F.Cu")
 		(net "+BATT")
 	)
 	(segment
-		(start 123.6 64.52)
-		(end 121.18 64.52)
-		(width 0.2)
+		(start 123.57 64.55)
+		(end 121.555761 64.55)
+		(width 0.3)
 		(layer "F.Cu")
 		(net "+BATT")
 	)
 	(segment
-		(start 120.6 66.9)
-		(end 121.175 67.475)
-		(width 0.2)
+		(start 123.6 64.52)
+		(end 123.57 64.55)
+		(width 0.3)
 		(layer "F.Cu")
 		(net "+BATT")
@@
 	)
 	(segment
-		(start 121.18 64.52)
-		(end 120.6 65.1)
-		(width 0.2)
+		(start 120.45 65.655761)
+		(end 120.45 66.3)
+		(width 0.3)
 		(layer "F.Cu")
 		(net "+BATT")
 	)
 	(segment
-		(start 120.6 65.1)
-		(end 120.6 66.9)
-		(width 0.2)
+		(start 120.45 66.3)
+		(end 121.625 67.475)
+		(width 0.3)
+		(layer "F.Cu")
+		(net "+BATT")
+	)
+	(segment
+		(start 121.555761 64.55)
+		(end 120.45 65.655761)
+		(width 0.3)
 		(layer "F.Cu")
 		(net "+BATT")
@@
 	)
 	(segment
+		(start 130.2 65.825)
+		(end 129.2 65.825)
+		(width 0.3)
+		(layer "F.Cu")
+		(net "GND")
+	)
+	(segment
 		(start 124.95 63.3)
 		(end 124.95 64.55)
@@
 	)
 	(segment
-		(start 129.025 65.65)
-		(end 129.2 65.825)
+		(start 135.81 64.6)
+		(end 135.81 63.8)
 		(width 0.3)
 		(layer "F.Cu")
@@
 	)
 	(segment
+		(start 121.1 65.925)
+		(end 122.1 65.925)
+		(width 0.3)
+		(layer "F.Cu")
+		(net "GND")
+	)
+	(segment
 		(start 124.95 64.55)
 		(end 125 64.6)
@@
 	)
 	(via
+		(at 130.2 65.825)
+		(size 0.6)
+		(drill 0.3)
+		(layers "F.Cu" "B.Cu")
+		(free yes)
+		(net "GND")
+	)
+	(via
 		(at 145.4 64.8)
 		(size 0.6)
@@
 	)
 	(via
-		(at 125 66)
+		(at 131 69.6)
+		(size 0.6)
+		(drill 0.3)
+		(layers "F.Cu" "B.Cu")
+		(free yes)
+		(net "GND")
+	)
+	(via
+		(at 131 71.2)
 		(size 0.6)
 		(drill 0.3)
 		(layers "F.Cu" "B.Cu")
+		(free yes)
 		(net "GND")
 	)
@@
 	)
 	(via
-		(at 125.7 64.6)
+		(at 121.1 65.925)
 		(size 0.6)
 		(drill 0.3)
 		(layers "F.Cu" "B.Cu")
+		(free yes)
 		(net "GND")
 	)
@@
 	)
 	(via
+		(at 118.2 74.4)
+		(size 0.6)
+		(drill 0.3)
+		(layers "F.Cu" "B.Cu")
+		(free yes)
+		(net "GND")
+	)
+	(via
 		(at 98.4 76.1)
 		(size 0.6)
@@
 	)
 	(via
-		(at 126.4 65.3)
+		(at 95.6 76.8)
 		(size 0.6)
 		(drill 0.3)
 		(layers "F.Cu" "B.Cu")
+		(free yes)
 		(net "GND")
 	)
 	(via
-		(at 95.6 76.8)
+		(at 118.2 69.2)
 		(size 0.6)
 		(drill 0.3)
@@
 	)
 	(via
+		(at 118.2 65.9)
+		(size 0.6)
+		(drill 0.3)
+		(layers "F.Cu" "B.Cu")
+		(free yes)
+		(net "GND")
+	)
+	(via
 		(at 96.3 63.9)
 		(size 0.6)
@@
 	)
 	(via
-		(at 125 64.6)
+		(at 146.8 64.8)
 		(size 0.6)
 		(drill 0.3)
 		(layers "F.Cu" "B.Cu")
+		(free yes)
 		(net "GND")
 	)
 	(via
-		(at 146.8 64.8)
+		(at 125.7 65.3)
 		(size 0.6)
 		(drill 0.3)
 		(layers "F.Cu" "B.Cu")
-		(free yes)
 		(net "GND")
 	)
@@
 	)
 	(via
-		(at 146.8 76.8)
+		(at 131 70.4)
 		(size 0.6)
 		(drill 0.3)
@@
 	)
 	(via
-		(at 146.8 64.1)
+		(at 146.8 76.8)
 		(size 0.6)
 		(drill 0.3)
@@
 	)
 	(via
-		(at 126.4 64.6)
+		(at 146.8 64.1)
 		(size 0.6)
 		(drill 0.3)
 		(layers "F.Cu" "B.Cu")
+		(free yes)
 		(net "GND")
 	)
 	(via
-		(at 126.4 66)
+		(at 118.2 65.1)
 		(size 0.6)
 		(drill 0.3)
 		(layers "F.Cu" "B.Cu")
+		(free yes)
 		(net "GND")
 	)
@@
 	)
 	(via
+		(at 124.95 65.3)
+		(size 0.6)
+		(drill 0.3)
+		(layers "F.Cu" "B.Cu")
+		(net "GND")
+	)
+	(via
+		(at 124.95 64.55)
+		(size 0.6)
+		(drill 0.3)
+		(layers "F.Cu" "B.Cu")
+		(net "GND")
+	)
+	(via
 		(at 97 63.2)
 		(size 0.6)
@@
 	)
 	(via
+		(at 125.7 66.05)
+		(size 0.6)
+		(drill 0.3)
+		(layers "F.Cu" "B.Cu")
+		(net "GND")
+	)
+	(via
+		(at 126.45 64.55)
+		(size 0.6)
+		(drill 0.3)
+		(layers "F.Cu" "B.Cu")
+		(net "GND")
+	)
+	(via
+		(at 118.2 64.3)
+		(size 0.6)
+		(drill 0.3)
+		(layers "F.Cu" "B.Cu")
+		(free yes)
+		(net "GND")
+	)
+	(via
+		(at 131 73.6)
+		(size 0.6)
+		(drill 0.3)
+		(layers "F.Cu" "B.Cu")
+		(free yes)
+		(net "GND")
+	)
+	(via
 		(at 123 63)
 		(size 0.6)
@@
 	)
 	(via
+		(at 118.2 70)
+		(size 0.6)
+		(drill 0.3)
+		(layers "F.Cu" "B.Cu")
+		(free yes)
+		(net "GND")
+	)
+	(via
 		(at 95.6 63.9)
 		(size 0.6)
@@
 	)
 	(via
-		(at 125.7 66)
+		(at 125.7 64.55)
 		(size 0.6)
 		(drill 0.3)
@@
 	)
 	(via
+		(at 118.2 73.6)
+		(size 0.6)
+		(drill 0.3)
+		(layers "F.Cu" "B.Cu")
+		(free yes)
+		(net "GND")
+	)
+	(via
 		(at 146.8 76.1)
 		(size 0.6)
@@
 	)
 	(via
+		(at 124.95 66.05)
+		(size 0.6)
+		(drill 0.3)
+		(layers "F.Cu" "B.Cu")
+		(net "GND")
+	)
+	(via
+		(at 131 72)
+		(size 0.6)
+		(drill 0.3)
+		(layers "F.Cu" "B.Cu")
+		(free yes)
+		(net "GND")
+	)
+	(via
+		(at 118.2 75.2)
+		(size 0.6)
+		(drill 0.3)
+		(layers "F.Cu" "B.Cu")
+		(free yes)
+		(net "GND")
+	)
+	(via
 		(at 144 76.8)
 		(size 0.6)
@@
 	)
 	(via
+		(at 131 72.8)
+		(size 0.6)
+		(drill 0.3)
+		(layers "F.Cu" "B.Cu")
+		(free yes)
+		(net "GND")
+	)
+	(via
 		(at 97.7 63.2)
 		(size 0.6)
@@
 	)
 	(via
-		(at 145.4 76.8)
+		(at 135.81 63.8)
 		(size 0.6)
 		(drill 0.3)
@@
 	)
 	(via
-		(at 125 65.3)
+		(at 126.45 66.05)
 		(size 0.6)
 		(drill 0.3)
@@
 	)
 	(via
-		(at 144.7 64.8)
+		(at 145.4 76.8)
 		(size 0.6)
 		(drill 0.3)
@@
 	)
 	(via
-		(at 125.7 65.3)
+		(at 118.2 70.8)
 		(size 0.6)
 		(drill 0.3)
 		(layers "F.Cu" "B.Cu")
+		(free yes)
+		(net "GND")
+	)
+	(via
+		(at 126.45 65.3)
+		(size 0.6)
+		(drill 0.3)
+		(layers "F.Cu" "B.Cu")
+		(net "GND")
+	)
+	(via
+		(at 144.7 64.8)
+		(size 0.6)
+		(drill 0.3)
+		(layers "F.Cu" "B.Cu")
+		(free yes)
 		(net "GND")
 	)
